File: Midi Stick.kicad_sch (KiCad schematic)
At the start: 36 parts, among them J1 USB 2.0 Type A Plug, J2 Aux, J3 ICSP, Q1 Mosfet N, X1 X1E0000210019

Commit message: WIP
Parts:
- removed C1, C2: 22pF, Capacitor_SMD:C_0603_1608Metric, symbol Midi Stick-altium-import:root_0_Cap
- removed C10, C8: 1uF, Capacitor_SMD:C_0603_1608Metric, symbol Midi Stick-altium-import:root_1_Cap
- removed C11: 10uF / ESR≤3Ω (Tantalum), Capacitor_SMD:C_1206_3216Metric, symbol Midi Stick-altium-import:root_1_Cap
- removed C12, C13, C4, C7, C9: 100nF, Capacitor_SMD:C_0603_1608Metric, symbol Midi Stick-altium-import:root_1_Cap
- removed C3: 4.7uF, Capacitor_SMD:C_0603_1608Metric, symbol Midi Stick-altium-import:root_1_Cap
- removed C5: 10uF, Capacitor_SMD:C_0603_1608Metric, symbol Midi Stick-altium-import:root_1_Cap
- removed J1: USB 2.0 Type A Plug, Connector_USB:USB_A_Molex_48037-2200_Horizontal, symbol Midi Stick-altium-import:root_0_mirrored_USB 2.0 Type A Plug
- removed MCU1: PIC32MX270F256B, Midi Stick:PIC32MX270F256B-I-SS_SSOP28_MC_MCH, symbol Midi Stick-altium-import:root_0_PIC32MX2xxFxxxB
- removed R10: 1k, Resistor_SMD:R_0603_1608Metric, symbol Midi Stick-altium-import:root_1_Resistor
- removed R8: 10k, Resistor_SMD:R_0603_1608Metric, symbol Midi Stick-altium-import:root_2_Resistor
- removed Reg1: 3.3V, Midi Stick:SOT229P700X180-4N, symbol Midi Stick-altium-import:root_0_VReg
- removed X1: X1E0000210019, Midi Stick:CRYSTAL-SMD_4P-L3.2-W2.5-BL-1, symbol CRYSTAL-SMD_4P-L3.2-W2.5-BL-1:X1E0000210019
- added C14, C18, C32: 10u, Capacitor_SMD:C_0805_2012Metric, symbol Device:C
- added C15, C16: 15p, Capacitor_SMD:C_0402_1005Metric, symbol Device:C
- added C17, C21, C24, C25, C26, C27, C28, C29, C30, C31: 100n, Capacitor_SMD:C_0402_1005Metric, symbol Device:C
- added C19, C20: 4.7u, RP2350_60QFN_minimal:C_0402_1005Metric_small_pads, symbol Device:C
- added C22, C23: 4.7u, Capacitor_SMD:C_0402_1005Metric, symbol Device:C
- added D7: PMEG6010ELR, Diode_SMD:D_SOD-123F, symbol Device:D_Schottky
- added H1, H2, H3, H4: MountingHole, MountingHole:MountingHole_2.7mm_M2.5, symbol Mechanical:MountingHole
- added J8: USB_C_Receptacle_USB2.0_16P, Connector_USB:USB_C_Receptacle_GCT_USB4105-xx-A_16P_TopMnt_Horizontal, symbol Connector:USB_C_Receptacle_USB2.0_16P
- added L1: 3.3u, RP2350_60QFN_minimal:L_pol_2016, symbol Device:L
- added R10, R8: 5k1, Resistor_SMD:R_0402_1005Metric, symbol Device:R
- added R11, R13: DNF, Resistor_SMD:R_0402_1005Metric, symbol Device:R
- added R12: 0, Resistor_SMD:R_0402_1005Metric, symbol Device:R
- added R14, R17: 1k, Resistor_SMD:R_0402_1005Metric, symbol Device:R
- added R16: 33, Resistor_SMD:R_0402_1005Metric, symbol Device:R
- added R18, R19: 27, Resistor_SMD:R_0402_1005Metric, symbol Device:R
- added SW1: SW_Push, Button_Switch_SMD:SW_Push_1P1T_NO_Vertical_Wuerth_434133025816, symbol Switch:SW_Push
- added U1: W25Q128JVS, Package_SO:SOIC-8_5.23x5.23mm_P1.27mm, symbol Memory_Flash:W25Q128JVS
- added U2: NCP1117-3.3_SOT223, Package_TO_SOT_SMD:SOT-223-3_TabPin2, symbol Regulator_Linear:NCP1117-3.3_SOT223
- added U3: RP2350_60QFN, RP2350_60QFN_minimal:RP2350-QFN-60-1EP_7x7_P0.4mm_EP3.4x3.4mm_ThermalVias, symbol MCU_RaspberryPi_RP2350:RP2350_60QFN
- added Y1: ABM8-272-T3, Crystal:Crystal_SMD_3225-4Pin_3.2x2.5mm, symbol Device:Crystal_GND24
Connections:
- net PGC is gone; now on net +3V3: J3.5
- net PGD is gone; now on net GND: J3.4
- net Aux: now also U3.8 (GPIO5)
- net Com LED: now also U3.28 (GPIO17)
- net GND: now also J3.2, C14.2, C15.2, C16.2, C17.2, C18.2, C19.2, C20.2, C21.2, C22.2, C23.2, C24.2, C25.2, C26.2, C27.2, C28.2, C29.2, C30.2, C31.2, C32.2, J8.A1 (GND), J8.A12 (GND), J8.B1 (GND), J8.B12 (GND), J8.S1 (SHIELD), R10.2, R8.2, SW1.1, U1.4 (GND), U2.1 (GND), U3.47 (VREG_PGND), U3.61 (GND), Y1.2, Y1.4; no longer J3.3
- net Out: now also U3.37 (GPIO25)
- net Power LED: now also U3.27 (GPIO16)
- net Signal LED: now also U3.29 (GPIO18)
- net +3.3V renamed +3V3
- net +3V3: now also C17.1, C18.1, C19.1, C25.1, C26.1, C27.1, C28.1, C29.1, C30.1, C31.1, C32.1, R13.1, R16.1, U1.8 (VCC), U2.2 (VO), U3.1 (IOVDD), U3.11 (IOVDD), U3.20 (IOVDD), U3.30 (IOVDD), U3.38 (IOVDD), U3.44 (ADC_AVDD), U3.45 (IOVDD), U3.49 (VREG_VIN), U3.53 (USB_OTP_VDD), U3.54 (QSPI_IOVDD); no longer J3.2
- net +5V renamed VBUS
- net VBUS: now also C14.1, D7.1 (K), U2.3 (VI)
- net D+ renamed USB_D+
- net USB_D+: now also J8.A6 (D+), J8.B6 (D+), R18.1
- net D- renamed USB_D-
- net USB_D-: now also J8.A7 (D-), J8.B7 (D-), R19.1
- net MCLR renamed SWCLK
- net SWCLK: now also U3.24 (SWCLK)
- new net: D7.2 (A), J8.A4 (VBUS), J8.A9 (VBUS), J8.B4 (VBUS), J8.B9 (VBUS)
- new net: J8.A5 (CC1), R8.1
- new net: J8.B5 (CC2), R10.1
- new net: C16.1, R14.2, Y1.3
- new net: R18.2, U3.52 (USB_DP)
- new net: R19.2, U3.51 (USB_DM)
- new net +1V1: C20.1, C21.1, C23.1, C24.1, L1.1, U3.23 (DVDD), U3.39 (DVDD), U3.50 (VREG_FB), U3.6 (DVDD)
- new net FLASH_SS: R11.2, R12.2, R13.2, U1.1 (~{CS})
- new net GPIO0: R11.1
- new net QSPI_SCLK: U1.6 (CLK), U3.56 (QSPI_SCLK)
- new net QSPI_SD0: U1.5 (DI(IO0)), U3.57 (QSPI_SD0)
- new net QSPI_SD1: U1.2 (DO(IO1)), U3.59 (QSPI_SD1)
- new net QSPI_SD2: U1.3 (IO2), U3.58 (QSPI_SD2)
- new net QSPI_SD3: U1.7 (IO3), U3.55 (QSPI_SD3)
- new net QSPI_SS: R12.1, R17.1, U3.60 (QSPI_SS)
- new net SWD: J3.3, U3.25 (SWD)
- new net VREG_AVDD: C22.1, R16.2, U3.46 (VREG_AVDD)
- new net VREG_LX: L1.2, U3.48 (VREG_LX)
- new net XIN: C15.1, U3.21 (XIN), Y1.1
- new net XOUT: R14.1, U3.22 (XOUT)
- new net ~{USB_BOOT}: R17.2, SW1.2
- no-connect marks 2 -> 28
Other:
- note added: "12MHz Crystal"
- note added: "Aux"
- note added: "Debug Connector"
- note added: "Flash"
- note added: "Make sure R7 and R8 are close to RP2350"
- note added: "Power"
- moved on the sheet: C6, D1, D2, D3, D4, D5, D6, J2, J3, Q1, R1, R2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

Commit message: WIP
Parts:
- removed H1, H2, H3, H4: MountingHole, MountingHole:MountingHole_2.7mm_M2.5, symbol Mechanical:MountingHole
- C19, C20: footprint RP2350_60QFN_minimal:C_0402_1005Metric_small_pads -> Capacitor_SMD:C_0402_1005Metric

Commit message: single sided
Parts:
- removed C6: 100nF, Capacitor_SMD:C_0603_1608Metric, symbol Midi Stick-altium-import:root_1_Cap
- removed D1: HFBR-141X, Midi Stick:HFBR-x41xZ, symbol Midi Stick-altium-import:root_0_HFBR-141X
- removed D6: TVS Diode, Diode_SMD:D_0603_1608Metric, symbol Midi Stick-altium-import:root_0_TVS Diode
- removed J2: Aux, Connector_PinSocket_2.54mm:PinSocket_1x02_P2.54mm_Vertical, symbol Midi Stick-altium-import:root_2_Header 2
- removed J3: ICSP, Connector_PinSocket_2.54mm:PinSocket_1x05_P2.54mm_Vertical, symbol Midi Stick-altium-import:root_0_Header 5
- removed Q1: Mosfet N, Midi Stick:SOT95P237X112-3N, symbol Midi Stick-altium-import:root_0_Mosfet N
- removed R1: 47Ohm, Resistor_SMD:R_0603_1608Metric, symbol Midi Stick-altium-import:root_1_Resistor
- removed R2, R3, R4: 1k, Resistor_SMD:R_0603_1608Metric, symbol Midi Stick-altium-import:root_1_Resistor
- removed R5: 470ohm, Resistor_SMD:R_0603_1608Metric, symbol Midi Stick-altium-import:root_0_Resistor
- removed R6: 10k, Resistor_SMD:R_0603_1608Metric, symbol Midi Stick-altium-import:root_1_Resistor
- removed R7: 1k, Resistor_SMD:R_0603_1608Metric, symbol Midi Stick-altium-import:root_2_Resistor
- removed R9: 150Ohm, Resistor_SMD:R_0603_1608Metric, symbol Midi Stick-altium-import:root_1_Resistor
- added C6: 100n, Capacitor_SMD:C_0402_1005Metric, symbol Device:C
- added J3: ICSP, Connector_PinSocket_2.54mm:PinSocket_1x07_P2.54mm_Vertical, symbol Connector_Generic:Conn_01x07
- added Q1: T2N7002AK, Package_TO_SOT_SMD:SOT-23, symbol Transistor_FET:T2N7002AK
- added R1: 470, Resistor_SMD:R_0402_1005Metric, symbol Device:R
- added R2, R3, R4, R7: 1k, Resistor_SMD:R_0402_1005Metric, symbol Device:R
- added R9: 150, Resistor_SMD:R_0402_1005Metric, symbol Device:R
- added TP1: Out Sense, TestPoint:TestPoint_Pad_1.0x1.0mm, symbol Connector:TestPoint
- added TP2: Out, Connector_PinHeader_2.54mm:PinHeader_1x01_P2.54mm_Vertical, symbol Connector:TestPoint
- added XT1: HFBR-1412, Midi Stick:HFBR-X41X, symbol HFBR-1412:HFBR-1412
Connections:
- net GPIO0 is gone; now on net UART0 TX: R11.1
- net +3V3: now also J3.7 (Pin_7)
- net Com LED: now also U3.41 (GPIO27_ADC1); no longer U3.28 (GPIO17)
- net GND: now also C6.2, J3.1 (Pin_1), Q1.2 (S), R7.2
- net Out: now also U3.15 (GPIO11), Q1.1 (G), R7.1, TP2.1; no longer U3.37 (GPIO25)
- net Out Sense: now also Q1.3 (D), R1.2, R9.2, TP1.1
- net Power LED: now also U3.40 (GPIO26_ADC0); no longer U3.27 (GPIO16)
- net SWCLK: now also J3.2 (Pin_2)
- net SWD: now also J3.3 (Pin_3)
- net Signal LED: now also U3.42 (GPIO28_ADC2); no longer U3.29 (GPIO18)
- net VBUS: now also D7.2 (A), J8.A4 (VBUS), J8.A9 (VBUS), J8.B4 (VBUS), J8.B9 (VBUS), C6.1, J3.6 (Pin_6), R2.1, R3.1, R4.1, XT1.2, XT1.7; no longer C14.1, D7.1 (K), U2.3 (VI)
- net at D3.1: now also R3.2
- net at D4.1: now also R4.2
- net at D2.1: now also R2.2
- net UART0 TX: now reaches U3.2 (GPIO0)
- net UART0 TX: now also J3.5 (Pin_5)
- net UART0 RX: now reaches U3.3 (GPIO1)
- net UART0 RX: now also J3.4 (Pin_4)
- net Aux: no longer names the net of U3.8 (GPIO5)
- new net: R9.1, XT1.6
- new net: C14.1, D7.1 (K), U2.3 (VI)
- new net: R1.1, XT1.3
Other:
- note removed: "Aux"
- moved on the sheet: C17, D2, D3, D4, R11, R12, R13, U1
