File: hardware/Midi Stick.kicad_pcb (KiCad board)
At the start: 2 copper layers, 57 x 19.9 mm, 54 parts, among them J3 ICSP, J8 USB_C_Receptacle_USB2.0_16P, Q1 T2N7002AK, SW1 SW_Push, U1 W25Q128JVS, U2 NCP1117-3.3_SOT223, U3 RP2350_60QFN, Y1 ABM8-272-T3

Commit message: Fix LED Power issue
Parts:
- R2, R3, R4: value 1k -> 470
Connections:
- R2 pad 1: VBUS -> +3V3
- R3 pad 1: VBUS -> +3V3
- R4 pad 1: VBUS -> +3V3
Routing:
- net VBUS: track 126.4 -> 116.5 mm
- net +3V3: track 113.5 -> 118.9 mm
