File: hardware/Midi Stick.kicad_sch (KiCad schematic)
At the start: 53 parts, among them J3 ICSP, J8 USB_C_Receptacle_USB2.0_16P, Q1 T2N7002AK, SW1 SW_Push, U1 W25Q128JVS, U2 NCP1117-3.3_SOT223, U3 RP2350_60QFN, Y1 ABM8-272-T3

Commit message: Fix LED Power issue
Parts:
- R2, R3, R4: value 1k -> 470
Connections:
- net +3V3: now also R2.1, R3.1, R4.1
- net VBUS: no longer R2.1, R3.1, R4.1
Other:
- moved on the sheet: C6, D2, D3, D4, Q1, R1, R2, R3, R4, R7, R9, TP1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
